File: Shifter/hardware/shifter.brd (EAGLE design)
At the start: 160 x 107.4 mm, 39 parts, among them J1 22-05-7078-07, J2 22-05-7038-03, J3 22-05-7028-02, J5 22-05-7028-02, J6 22-05-7028-02

Commit message: no message
Parts:
- C4, C5: value (none) -> 0.33u
- F1: value (none) -> 1A
- Q1, Q2, Q3, Q4, Q5: value (none) -> 2N7000
- R1, R10, R12, R14, R15, R17, R2, R3, R4, R5, R6, R7, R8, R9: value (none) -> 10k
- R11, R13: value (none) -> 14k
- moved JP4 0.25 mm to (56.9, 68.6)
Other:
- board text added: "Shifter Vulcanix - EPSA 2017/2018"
