File: Tableau/Carte commande/tableau.sch (EAGLE design)
At the start: 42 parts, among them IC1 74LS47N, IC3 74LS47N, IC4 74LS47N, IC5 LM3914N, IC6 LM2576T

Commit message: no message
Parts:
- removed C8: (no value), rcl:C-EU025-030X050
- removed X2: (no value), con-molex:KK-156-2
- added LED3, LED4: VERT, led:LED3MM
- added R6, R7: (no value), resistor:R-EU_0204/7
- D1: value (none) -> 1N5822
- L1: value (none) -> 100uH
- R1: value (none) -> 10k
Connections:
- removed net USB_D+: PIC18F25K80.RC5/SDO, X2-2.S
- removed net USB_D-: PIC18F25K80.RC4/SDI/SDA, X2-1.S
- new net LED_1: PIC18F25K80.RC5/SDO, R7.1
- new net LED_2: PIC18F25K80.RC4/SDI/SDA, R6.1
- new net N$38: LED3.A, R6.2
- new net N$39: LED4.A, R7.2
- net GND: now also LED3.C, LED4.C; no longer C8.1
- net MCLR: no longer C8.2
Changed lines of the file:
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@@
 <part name="R4" library="resistor" deviceset="R-EU_" device="0204/7"/>
 <part name="GND8" library="supply1" deviceset="GND" device=""/>
-<part name="R1" library="resistor" deviceset="R-EU_" device="0204/7"/>
+<part name="R1" library="resistor" deviceset="R-EU_" device="0204/7" value="10k"/>
 <part name="GND1" library="supply1" deviceset="GND" device=""/>
 <part name="P+4" library="supply1" deviceset="VCC" device=""/>
@@
 <part name="GND18" library="supply1" deviceset="GND" device=""/>
 <part name="FRAME1" library="bmp180module" deviceset="FRAME_A3" device=""/>
-<part name="C8" library="rcl" deviceset="C-EU" device="025-030X050"/>
 <part name="X9" library="con-molex" deviceset="KK-156-5" device=""/>
 <part name="GND19" library="supply1" deviceset="GND" device=""/>
@@
 <part name="P+12" library="supply1" deviceset="VCC" device=""/>
 <part name="X8" library="con-molex" library_urn="urn:adsk.eagle:library:165" deviceset="KK-156-3" device=""/>
-<part name="X2" library="con-molex" library_urn="urn:adsk.eagle:library:165" deviceset="KK-156-2" device=""/>
 <part name="X7" library="con-molex" library_urn="urn:adsk.eagle:library:165" deviceset="KK-156-2" device=""/>
-<part name="D1" library="diode" library_urn="urn:adsk.eagle:library:210" deviceset="SCHOTTKY-DIODE" device="DO201T15" package3d_urn="urn:adsk.eagle:package:43354/1"/>
-<part name="L1" library="WE-TI" deviceset="WE-TI" device="_8012B" technology="-744743102"/>
+<part name="D1" library="diode" library_urn="urn:adsk.eagle:library:210" deviceset="SCHOTTKY-DIODE" device="DO201T15" package3d_urn="urn:adsk.eagle:package:43354/1" value="1N5822"/>
+<part name="L1" library="WE-TI" deviceset="WE-TI" device="_8012B" technology="-744743102" value="100uH"/>
 <part name="X10" library="con-molex" library_urn="urn:adsk.eagle:library:165" deviceset="KK-156-2" device=""/>
 <part name="R2" library="resistor" deviceset="R-EU_" device="0204/7"/>
@@
 <part name="X5" library="con-molex" library_urn="urn:adsk.eagle:library:165" deviceset="KK-156-2" device=""/>
 <part name="R5" library="resistor" deviceset="R-EU_" device="0204/7" value="120"/>
+<part name="R6" library="resistor" deviceset="R-EU_" device="0204/7"/>
+<part name="R7" library="resistor" deviceset="R-EU_" device="0204/7"/>
+<part name="LED3" library="led" deviceset="LED" device="3MM" value="VERT"/>
+<part name="LED4" library="led" deviceset="LED" device="3MM" value="VERT"/>
+<part name="GND17" library="supply1" deviceset="GND" device=""/>
 </parts>
 <sheets>
@@
 <instance part="GND18" gate="1" x="-12.7" y="-78.74" rot="R270"/>
 <instance part="FRAME1" gate="G$1" x="-180.34" y="-106.68"/>
-<instance part="C8" gate="G$1" x="-2.54" y="73.66" rot="R180"/>
 <instance part="X9" gate="-1" x="78.74" y="132.08"/>
 <instance part="X9" gate="-2" x="78.74" y="129.54"/>
@@
 <instance part="X8" gate="-2" x="-50.8" y="-35.56"/>
 <instance part="X8" gate="-3" x="-50.8" y="-38.1"/>
-<instance part="X2" gate="-1" x="137.16" y="142.24"/>
-<instance part="X2" gate="-2" x="137.16" y="137.16"/>
 <instance part="X7" gate="-1" x="-147.32" y="66.04"/>
 <instance part="X7" gate="-2" x="-147.32" y="60.96"/>
@@
 <instance part="X5" gate="-2" x="33.02" y="-48.26"/>
 <instance part="R5" gate="G$1" x="-88.9" y="-40.64" rot="R90"/>
+<instance part="R6" gate="G$1" x="-104.14" y="20.32"/>
+<instance part="R7" gate="G$1" x="-104.14" y="10.16"/>
+<instance part="LED3" gate="G$1" x="-93.98" y="20.32" rot="R90"/>
+<instance part="LED4" gate="G$1" x="-93.98" y="10.16" rot="R90"/>
+<instance part="GND17" gate="1" x="-78.74" y="10.16" rot="R90"/>
 </instances>
 <busses>
@@
 <segment>
 <pinref part="GND1" gate="1" pin="GND"/>
-<wire x1="-15.24" y1="63.5" x2="-15.24" y2="66.04" width="0.1524" layer="91"/>
 <pinref part="SW1" gate="G$1" pin="P$1"/>
-<pinref part="C8" gate="G$1" pin="1"/>
-<wire x1="-15.24" y1="66.04" x2="-15.24" y2="68.58" width="0.1524" layer="91"/>
-<wire x1="-2.54" y1="71.12" x2="-2.54" y2="66.04" width="0.1524" layer="91"/>
-<wire x1="-2.54" y1="66.04" x2="-15.24" y2="66.04" width="0.1524" layer="91"/>
-<junction x="-15.24" y="66.04"/>
+<wire x1="-15.24" y1="63.5" x2="-15.24" y2="68.58" width="0.1524" layer="91"/>
 </segment>
 <segment>
@@
 <wire x1="-60.96" y1="-35.56" x2="-53.34" y2="-35.56" width="0.1524" layer="91"/>
 </segment>
+<segment>
+<pinref part="LED3" gate="G$1" pin="C"/>
+<wire x1="-88.9" y1="20.32" x2="-86.36" y2="20.32" width="0.1524" layer="91"/>
+<wire x1="-86.36" y1="20.32" x2="-86.36" y2="10.16" width="0.1524" layer="91"/>
+<pinref part="LED4" gate="G$1" pin="C"/>
+<wire x1="-86.36" y1="10.16" x2="-88.9" y2="10.16" width="0.1524" layer="91"/>
+<wire x1="-86.36" y1="10.16" x2="-81.28" y2="10.16" width="0.1524" layer="91"/>
+<pinref part="GND17" gate="1" pin="GND"/>
+<junction x="-86.36" y="10.16"/>
+</segment>
 </net>
 <net name="CAN_RX" class="0">
@@
 <label x="-17.78" y="81.28" size="1.778" layer="95" rot="R180" xref="yes"/>
 <pinref part="SW1" gate="G$1" pin="P$2"/>
-<pinref part="C8" gate="G$1" pin="2"/>
-<wire x1="-2.54" y1="78.74" x2="-2.54" y2="81.28" width="0.1524" layer="91"/>
-<wire x1="-2.54" y1="81.28" x2="-15.24" y2="81.28" width="0.1524" layer="91"/>
 </segment>
 <segment>
@@
 </segment>
 </net>
-<net name="USB_D+" class="0">
+<net name="LED_2" class="0">
+<segment>
+<pinref part="PIC18F25K80" gate="G$1" pin="RC4/SDI/SDA"/>
+<wire x1="99.06" y1="68.58" x2="101.6" y2="68.58" width="0.1524" layer="91"/>
+<wire x1="101.6" y1="68.58" x2="101.6" y2="60.96" width="0.1524" layer="91"/>
+<label x="101.6" y="60.96" size="1.778" layer="95" xref="yes"/>
+</segment>
+<segment>
+<pinref part="R6" gate="G$1" pin="1"/>
+<wire x1="-109.22" y1="20.32" x2="-111.76" y2="20.32" width="0.1524" layer="91"/>
+<label x="-111.76" y="20.32" size="1.778" layer="95" rot="R180" xref="yes"/>
+</segment>
+</net>
+<net name="LED_1" class="0">
 <segment>
 <pinref part="PIC18F25K80" gate="G$1" pin="RC5/SDO"/>
@@
 </segment>
 <segment>
-<pinref part="X2" gate="-2" pin="S"/>
-<wire x1="134.62" y1="137.16" x2="132.08" y2="137.16" width="0.1524" layer="91"/>
-<label x="132.08" y="137.16" size="1.778" layer="95" rot="R180" xref="yes"/>
-</segment>
-</net>
-<net name="USB_D-" class="0">
-<segment>
-<pinref part="PIC18F25K80" gate="G$1" pin="RC4/SDI/SDA"/>
-<wire x1="99.06" y1="68.58" x2="101.6" y2="68.58" width="0.1524" layer="91"/>
-<wire x1="101.6" y1="68.58" x2="101.6" y2="60.96" width="0.1524" layer="91"/>
-<label x="101.6" y="60.96" size="1.778" layer="95" xref="yes"/>
-</segment>
-<segment>
-<pinref part="X2" gate="-1" pin="S"/>
-<wire x1="134.62" y1="142.24" x2="132.08" y2="142.24" width="0.1524" layer="91"/>
-<label x="132.08" y="142.24" size="1.778" layer="95" rot="R180" xref="yes"/>
+<pinref part="R7" gate="G$1" pin="1"/>
+<wire x1="-109.22" y1="10.16" x2="-111.76" y2="10.16" width="0.1524" layer="91"/>
+<label x="-111.76" y="10.16" size="1.778" layer="95" rot="R180" xref="yes"/>
+</segment>
+</net>
+<net name="N$38" class="0">
+<segment>
+<pinref part="R6" gate="G$1" pin="2"/>
+<pinref part="LED3" gate="G$1" pin="A"/>
+<wire x1="-99.06" y1="20.32" x2="-96.52" y2="20.32" width="0.1524" layer="91"/>
+</segment>
+</net>
+<net name="N$39" class="0">
+<segment>
+<pinref part="R7" gate="G$1" pin="2"/>
+<pinref part="LED4" gate="G$1" pin="A"/>
+<wire x1="-99.06" y1="10.16" x2="-96.52" y2="10.16" width="0.1524" layer="91"/>
 </segment>
 </net>
@@
 </sheet>
 </sheets>
+<errors>
+</errors>
 </schematic>
 </drawing>
